File: Desenvolvimento_IC2S-EBM2-2609-V5.0/Projeto_IC2S-EBM2-2609-V5.0/03_alimentacao.kicad_sch (KiCad schematic)
At the start: 21 parts, among them U1 TPS7A4001DGN, U2 ADR4525WBRZ-R7, U3 TL431B, U4 MCP1824T-3302E/OT

Commit message: Revisao de 28-09 (vinda da EBM7): ramo unico de 24 V, 100 nF a 50 V, um so MPN de 1 uF
- Saem F1 (250 mA), D3 e R3: o F1 nao aguenta o arranque da placa toda e o R3
  so existia para o limitar. F2 + D4 alimentam o U1 e os lacos; +24V_REG passa
  a +24V_ADC. C1 fica (Cin do TPS7A4001). Esquematico e PCB (sem pistas).
- 100 nF fora do 24 V -> TDK C1608X7R1H104K080AA (50 V); C29 (+24V_ADC) fica
  GRM188R72A104KA35D (100 V). 1 uF -> TDK C1608X7R1H105K080AB.
- Folha 2 notas 3, 11, 13 e 14; BOM preliminar regenerada; README, registo e
  lista de datasheets. Alteracao posterior ao Portao 1, registada como tal.

Co-Authored-By: Claude Opus 5.5 (1M context) <noreply@anthropic.com>
Claude-Session: https://claude.ai/code/session_01KPnkiJQKrkjgRqqw9M78ie
Parts:
- C3, C6, C9: value 100nF -> 100nF/50V; MPN GRM188R72A104KA35D -> C1608X7R1H104K080AA
Connections:
- net +24V_REG renamed +24V_ADC
Changed lines of the file:
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@@
 			)
 		)
-		(property "Value" "100nF"
+		(property "Value" "100nF/50V"
 			(at 193.04 66.04 0)
 			(show_name no)
@@
 			)
 		)
-		(property "MPN" "GRM188R72A104KA35D"
+		(property "MPN" "C1608X7R1H104K080AA"
 			(at 190.5 64.77 0)
 			(hide yes)
@@
 			)
 		)
-		(property "Value" "+24V_REG"
+		(property "Value" "+24V_ADC"
 			(at 33.02 57.15 0)
 			(show_name no)
@@
 			)
 		)
-		(property "Value" "100nF"
+		(property "Value" "100nF/50V"
 			(at 99.06 71.12 0)
 			(show_name no)
@@
 			)
 		)
-		(property "MPN" "GRM188R72A104KA35D"
+		(property "MPN" "C1608X7R1H104K080AA"
 			(at 96.52 69.85 0)
 			(hide yes)
@@
 			)
 		)
-		(property "Value" "100nF"
+		(property "Value" "100nF/50V"
 			(at 40.64 121.92 0)
 			(show_name no)
@@
 			)
 		)
-		(property "MPN" "GRM188R72A104KA35D"
+		(property "MPN" "C1608X7R1H104K080AA"
 			(at 38.1 120.65 0)
 			(hide yes)
