File: Desenvolvimento_IC2S-EBM2-2609-V5.0/Projeto_IC2S-EBM2-2609-V5.0/06_lacos.kicad_sch (KiCad schematic)
At the start: 81 parts, among them U10 TPS26613DDFR, U11 TPS26613DDFR, U12 TPS26613DDFR, U13 TPS26613DDFR, U14 TPS7A4001DGN, U8 TPS26613DDFR, U9 TPS26613DDFR

Commit message: Revisao de 28-09 (vinda da EBM7): ramo unico de 24 V, 100 nF a 50 V, um so MPN de 1 uF
- Saem F1 (250 mA), D3 e R3: o F1 nao aguenta o arranque da placa toda e o R3
  so existia para o limitar. F2 + D4 alimentam o U1 e os lacos; +24V_REG passa
  a +24V_ADC. C1 fica (Cin do TPS7A4001). Esquematico e PCB (sem pistas).
- 100 nF fora do 24 V -> TDK C1608X7R1H104K080AA (50 V); C29 (+24V_ADC) fica
  GRM188R72A104KA35D (100 V). 1 uF -> TDK C1608X7R1H105K080AB.
- Folha 2 notas 3, 11, 13 e 14; BOM preliminar regenerada; README, registo e
  lista de datasheets. Alteracao posterior ao Portao 1, registada como tal.

Co-Authored-By: Claude Opus 5.5 (1M context) <noreply@anthropic.com>
Claude-Session: https://claude.ai/code/session_01KPnkiJQKrkjgRqqw9M78ie
Parts:
- C17, C18, C19, C20, C21, C22, C34: value 100nF/100V -> 100nF/50V; MPN GRM188R72A104KA35D -> C1608X7R1H104K080AA
- C23, C24, C25, C26, C27, C28: value 100nF -> 100nF/50V; MPN GRM188R72A104KA35D -> C1608X7R1H104K080AA
Changed lines of the file:
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@@
 			)
 		)
-		(property "Value" "100nF/100V"
+		(property "Value" "100nF/50V"
 			(at 63.5 62.23 0)
 			(show_name no)
@@
 			)
 		)
-		(property "MPN" "GRM188R72A104KA35D"
+		(property "MPN" "C1608X7R1H104K080AA"
 			(at 60.96 60.96 0)
 			(hide yes)
@@
 			)
 		)
-		(property "Value" "100nF"
+		(property "Value" "100nF/50V"
 			(at 99.06 81.28 0)
 			(show_name no)
@@
 			)
 		)
-		(property "MPN" "GRM188R72A104KA35D"
+		(property "MPN" "C1608X7R1H104K080AA"
 			(at 96.52 80.01 0)
 			(hide yes)
@@
 			)
 		)
-		(property "Value" "100nF/100V"
+		(property "Value" "100nF/50V"
 			(at 63.5 123.19 0)
 			(show_name no)
@@
 			)
 		)
-		(property "MPN" "GRM188R72A104KA35D"
+		(property "MPN" "C1608X7R1H104K080AA"
 			(at 60.96 121.92 0)
 			(hide yes)
@@
 			)
 		)
-		(property "Value" "100nF"
+		(property "Value" "100nF/50V"
 			(at 99.06 142.24 0)
 			(show_name no)
@@
 			)
 		)
-		(property "MPN" "GRM188R72A104KA35D"
+		(property "MPN" "C1608X7R1H104K080AA"
 			(at 96.52 140.97 0)
 			(hide yes)
@@
 			)
 		)
-		(property "Value" "100nF/100V"
+		(property "Value" "100nF/50V"
 			(at 63.5 184.15 0)
 			(show_name no)
@@
 			)
 		)
-		(property "MPN" "GRM188R72A104KA35D"
+		(property "MPN" "C1608X7R1H104K080AA"
 			(at 60.96 182.88 0)
 			(hide yes)
@@
 			)
 		)
-		(property "Value" "100nF"
+		(property "Value" "100nF/50V"
 			(at 99.06 203.2 0)
 			(show_name no)
@@
 			)
 		)
-		(property "MPN" "GRM188R72A104KA35D"
+		(property "MPN" "C1608X7R1H104K080AA"
 			(at 96.52 201.93 0)
 			(hide yes)
@@
 			)
 		)
-		(property "Value" "100nF/100V"
+		(property "Value" "100nF/50V"
 			(at 200.66 62.23 0)
 			(show_name no)
@@
 			)
 		)
-		(property "MPN" "GRM188R72A104KA35D"
+		(property "MPN" "C1608X7R1H104K080AA"
 			(at 198.12 60.96 0)
 			(hide yes)
@@
 			)
 		)
-		(property "Value" "100nF"
+		(property "Value" "100nF/50V"
 			(at 236.22 81.28 0)
 			(show_name no)
@@
 			)
 		)
-		(property "MPN" "GRM188R72A104KA35D"
+		(property "MPN" "C1608X7R1H104K080AA"
 			(at 233.68 80.01 0)
 			(hide yes)
@@
 			)
 		)
-		(property "Value" "100nF/100V"
+		(property "Value" "100nF/50V"
 			(at 200.66 123.19 0)
 			(show_name no)
@@
 			)
 		)
-		(property "MPN" "GRM188R72A104KA35D"
+		(property "MPN" "C1608X7R1H104K080AA"
 			(at 198.12 121.92 0)
 			(hide yes)
@@
 			)
 		)
-		(property "Value" "100nF"
+		(property "Value" "100nF/50V"
 			(at 236.22 142.24 0)
 			(show_name no)
@@
 			)
 		)
-		(property "MPN" "GRM188R72A104KA35D"
+		(property "MPN" "C1608X7R1H104K080AA"
 			(at 233.68 140.97 0)
 			(hide yes)
@@
 			)
 		)
-		(property "Value" "100nF/100V"
+		(property "Value" "100nF/50V"
 			(at 200.66 184.15 0)
 			(show_name no)
@@
 			)
 		)
-		(property "MPN" "GRM188R72A104KA35D"
+		(property "MPN" "C1608X7R1H104K080AA"
 			(at 198.12 182.88 0)
 			(hide yes)
@@
 			)
 		)
-		(property "Value" "100nF"
+		(property "Value" "100nF/50V"
 			(at 236.22 203.2 0)
 			(show_name no)
@@
 			)
 		)
-		(property "MPN" "GRM188R72A104KA35D"
+		(property "MPN" "C1608X7R1H104K080AA"
 			(at 233.68 201.93 0)
 			(hide yes)
@@
 			)
 		)
-		(property "Value" "100nF/100V"
+		(property "Value" "100nF/50V"
 			(at 218.44 256.54 0)
 			(show_name no)
@@
 			)
 		)
-		(property "MPN" "GRM188R72A104KA35D"
+		(property "MPN" "C1608X7R1H104K080AA"
 			(at 215.9 255.27 0)
 			(hide yes)
