File: Desenvolvimento_IC2S-EBM2-2609-V5.0/Projeto_IC2S-EBM2-2609-V5.0/04_barreira.kicad_sch (KiCad schematic)
At the start: 8 parts, among them U5 MCP1824ST-3302E/DB, U6 ISO7141CCDBQR

Commit message: Revisao de 28-09 (vinda da EBM7): ramo unico de 24 V, 100 nF a 50 V, um so MPN de 1 uF
- Saem F1 (250 mA), D3 e R3: o F1 nao aguenta o arranque da placa toda e o R3
  so existia para o limitar. F2 + D4 alimentam o U1 e os lacos; +24V_REG passa
  a +24V_ADC. C1 fica (Cin do TPS7A4001). Esquematico e PCB (sem pistas).
- 100 nF fora do 24 V -> TDK C1608X7R1H104K080AA (50 V); C29 (+24V_ADC) fica
  GRM188R72A104KA35D (100 V). 1 uF -> TDK C1608X7R1H105K080AB.
- Folha 2 notas 3, 11, 13 e 14; BOM preliminar regenerada; README, registo e
  lista de datasheets. Alteracao posterior ao Portao 1, registada como tal.

Co-Authored-By: Claude Opus 5.5 (1M context) <noreply@anthropic.com>
Claude-Session: https://claude.ai/code/session_01KPnkiJQKrkjgRqqw9M78ie
Parts:
- C10: value 1uF -> 1uF/50V; MPN C0603C105K4RACTU -> C1608X7R1H105K080AB
- C12, C13: value 100nF -> 100nF/50V; MPN GRM188R72A104KA35D -> C1608X7R1H104K080AA
Changed lines of the file:
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@@
 			)
 		)
-		(property "Value" "1uF"
+		(property "Value" "1uF/50V"
 			(at 68.58 71.12 0)
 			(show_name no)
@@
 			)
 		)
-		(property "MPN" "C0603C105K4RACTU"
+		(property "MPN" "C1608X7R1H105K080AB"
 			(at 71.12 69.85 0)
 			(hide yes)
@@
 			)
 		)
-		(property "Value" "100nF"
+		(property "Value" "100nF/50V"
 			(at 114.3 71.12 0)
 			(show_name no)
@@
 			)
 		)
-		(property "MPN" "GRM188R72A104KA35D"
+		(property "MPN" "C1608X7R1H104K080AA"
 			(at 111.76 69.85 0)
 			(hide yes)
@@
 			)
 		)
-		(property "Value" "100nF"
+		(property "Value" "100nF/50V"
 			(at 165.1 71.12 0)
 			(show_name no)
@@
 			)
 		)
-		(property "MPN" "GRM188R72A104KA35D"
+		(property "MPN" "C1608X7R1H104K080AA"
 			(at 162.56 69.85 0)
 			(hide yes)

Commit message: LDO 3,3 V do lado PLC: U5 MCP1824ST (SOT-223) -> MCP1824T-3302E/OT (SOT-23-5), mesmo MPN do U4
- Criterio da equipa: menos MPN, mais pecas do mesmo tipo; o MCP1824ST sai.
- SHDN a VIN, PG aberto; mesmo datasheet (DS22070A), estavel com ceramico >= 1 uF.
- Esquematico: ERC 0; netlist so muda os pinos do U5. PCB: pegada SOT-23-5 no
  mesmo sitio; placa ainda sem pistas; nota 3 da folha 4 actualizada.
- Registo: alteracao_LDO_3V3_lado_PLC_2026-09-28.md (comparacao, verificacao e
  riscos em aberto). BOM e PDF do esquematico regenerados.

Co-Authored-By: Claude Opus 5.5 (1M context) <noreply@anthropic.com>
Claude-Session: https://claude.ai/code/session_01KPnkiJQKrkjgRqqw9M78ie
Parts:
- U5: value MCP1824ST-3302E/DB -> MCP1824T-3302E/OT; footprint EBM2_V5:SOT-223-3 -> EBM2_V5:SOT-23-5; symbol EBM2_V5:MCP1824ST-3302E -> EBM2_V5:MCP1824T-3302E_OT; MPN MCP1824ST-3302E/DB -> MCP1824T-3302E/OT
Connections:
- net +3.3V_DIG: now also U5.5 (OUT); no longer U5.3 (VOUT)
- net +5V: now also U5.3 (~{SHDN})
- net DGND: no longer U5.4 (TAB)
- no-connect marks 0 -> 1
Other:
- note added: "3. U5 MCP1824T-3302E/OT SOT-23-5 (28-09-2026, era MCP1824S SOT-223): mesmo MPN do U4; pinos pag. 2 do DS22070A;"
- note added: "entrada 2,1-6,0 V; estavel com >= 1 uF ceramico (pag. 1); C11 = 2,2 uF. SHDN a VIN, PG aberto."
- note removed: "3. U5 MCP1824S SOT-223-3: pinos na figura da pag. 2 do DS22070A. Entrada 2,1-6,0 V;"
- note removed: "estavel com >= 1 uF ceramico (pag. 1); C11 = 2,2 uF (rev. 2.5). Sem enable: EN1 e do isolador."
Changed lines of the file:
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@@
 	(wire
 		(pts
-			(xy 83.82 71.12) (xy 86.36 71.12)
+			(xy 99.06 66.04) (xy 101.6 66.04)
 		)
 		(stroke
@@
 	(wire
 		(pts
-			(xy 86.36 71.12) (xy 88.9 71.12)
+			(xy 101.6 66.04) (xy 111.76 66.04)
 		)
 		(stroke
@@
 	(wire
 		(pts
-			(xy 99.06 66.04) (xy 101.6 66.04)
+			(xy 111.76 66.04) (xy 116.84 66.04)
 		)
 		(stroke
@@
 	(wire
 		(pts
-			(xy 101.6 66.04) (xy 111.76 66.04)
+			(xy 129.54 80.01) (xy 124.46 80.01)
 		)
 		(stroke
@@
 	(wire
 		(pts
-			(xy 111.76 66.04) (xy 116.84 66.04)
+			(xy 129.54 82.55) (xy 124.46 82.55)
 		)
 		(stroke
@@
 	(wire
 		(pts
-			(xy 129.54 80.01) (xy 124.46 80.01)
+			(xy 129.54 95.25) (xy 124.46 95.25)
 		)
 		(stroke
@@
 	(wire
 		(pts
-			(xy 129.54 82.55) (xy 124.46 82.55)
+			(xy 129.54 97.79) (xy 124.46 97.79)
 		)
 		(stroke
@@
 	(wire
 		(pts
-			(xy 129.54 95.25) (xy 124.46 95.25)
+			(xy 149.86 80.01) (xy 157.48 80.01)
 		)
 		(stroke
@@
 	(wire
 		(pts
-			(xy 129.54 97.79) (xy 124.46 97.79)
+			(xy 157.48 80.01) (xy 157.48 66.04)
 		)
 		(stroke
@@
 	(wire
 		(pts
-			(xy 149.86 80.01) (xy 157.48 80.01)
+			(xy 157.48 66.04) (xy 160.02 66.04)
 		)
 		(stroke
@@
 	(wire
 		(pts
-			(xy 157.48 80.01) (xy 157.48 66.04)
+			(xy 160.02 66.04) (xy 162.56 66.04)
 		)
 		(stroke
@@
 	(wire
 		(pts
-			(xy 157.48 66.04) (xy 160.02 66.04)
+			(xy 162.56 66.04) (xy 170.18 66.04)
 		)
 		(stroke
@@
 	(wire
 		(pts
-			(xy 160.02 66.04) (xy 162.56 66.04)
+			(xy 149.86 95.25) (xy 154.94 95.25)
 		)
 		(stroke
@@
 	(wire
 		(pts
-			(xy 162.56 66.04) (xy 170.18 66.04)
+			(xy 177.8 66.04) (xy 187.96 66.04)
 		)
 		(stroke
@@
 	(wire
 		(pts
-			(xy 149.86 95.25) (xy 154.94 95.25)
+			(xy 149.86 82.55) (xy 154.94 82.55)
 		)
 		(stroke
@@
 	(wire
 		(pts
-			(xy 177.8 66.04) (xy 187.96 66.04)
+			(xy 149.86 97.79) (xy 154.94 97.79)
 		)
 		(stroke
@@
 		)
 	)
-	(wire
-		(pts
-			(xy 149.86 82.55) (xy 154.94 82.55)
-		)
-		(stroke
-			(width 0)
-			(type default)
-		)
-	)
-	(wire
-		(pts
-			(xy 149.86 97.79) (xy 154.94 97.79)
-		)
-		(stroke
-			(width 0)
-			(type default)
-		)
-	)
 	(junction
 		(at 71.12 66.04)
-		(diameter 0)
-		(color 0 0 0 0)
-	)
-	(junction
-		(at 86.36 71.12)
 		(diameter 0)
 		(color 0 0 0 0)
@@
 		)
 	)
-	(text "3. U5 MCP1824S SOT-223-3: pinos na figura da pag. 2 do DS22070A. Entrada 2,1-6,0 V;"
+	(text "3. U5 MCP1824T-3302E/OT SOT-23-5 (28-09-2026, era MCP1824S SOT-223): mesmo MPN do U4; pinos pag. 2 do DS22070A;"
 		(exclude_from_sim no)
 		(at 25.4 147.32 0)
@@
 		)
 	)
-	(text "   estavel com >= 1 uF ceramico (pag. 1); C11 = 2,2 uF (rev. 2.5). Sem enable: EN1 e do isolador."
+	(text "   entrada 2,1-6,0 V; estavel com >= 1 uF ceramico (pag. 1); C11 = 2,2 uF. SHDN a VIN, PG aberto."
 		(exclude_from_sim no)
 		(at 25.4 151.13 0)
@@
 	)
 	(symbol
-		(lib_id "EBM2_V5:MCP1824ST-3302E")
-		(at 86.36 66.04 0)
+		(lib_id "EBM2_V5:MCP1824T-3302E_OT")
+		(at 86.36 68.58 0)
 		(unit 1)
 		(body_style 1)
@@
 			)
 		)
-		(property "Value" "MCP1824ST-3302E/DB"
+		(property "Value" "MCP1824T-3302E/OT"
 			(at 86.36 59.69 0)
 			(show_name no)
@@
 			)
 		)
-		(property "Footprint" "EBM2_V5:SOT-223-3"
+		(property "Footprint" "EBM2_V5:SOT-23-5"
 			(at 86.36 66.04 0)
 			(hide yes)
@@
 			)
 		)
-		(property "MPN" "MCP1824ST-3302E/DB"
+		(property "MPN" "MCP1824T-3302E/OT"
 			(at 86.36 66.04 0)
 			(hide yes)
@@
 		)
 		(pin "4"
+		)
+		(pin "5"
 		)
 		(instances
@@
 	(symbol
 		(lib_id "power:GND")
-		(at 86.36 71.12 0)
+		(at 86.36 76.2 0)
 		(unit 1)
 		(body_style 1)
@@
 		(dnp no)
 		(property "Reference" "#PWR403"
-			(at 86.36 71.12 0)
+			(at 86.36 76.2 0)
 			(hide yes)
 			(show_name no)
@@
 		)
 		(property "Value" "DGND"
-			(at 86.36 74.93 0)
+			(at 86.36 80.01 0)
 			(show_name no)
 			(do_not_autoplace no)
@@
 		)
 		(property "Footprint" ""
-			(at 86.36 71.12 0)
+			(at 86.36 76.2 0)
 			(hide yes)
 			(show_name no)
@@
 		)
 		(property "Datasheet" ""
-			(at 86.36 71.12 0)
+			(at 86.36 76.2 0)
 			(hide yes)
 			(show_name no)
@@
 		)
 		(property "Description" ""
-			(at 86.36 71.12 0)
+			(at 86.36 76.2 0)
 			(hide yes)
 			(show_name no)
@@
 	)
 	(embedded_fonts no)
+	(wire
+		(pts
+			(xy 73.66 66.04) (xy 77.47 66.04)
+		)
+		(stroke
+			(width 0)
+			(type default)
+		)
+	)
+	(wire
+		(pts
+			(xy 77.47 66.04) (xy 78.74 66.04)
+		)
+		(stroke
+			(width 0)
+			(type default)
+		)
+	)
+	(wire
+		(pts
+			(xy 78.74 68.58) (xy 77.47 68.58)
+		)
+		(stroke
+			(width 0)
+			(type default)
+		)
+	)
+	(wire
+		(pts
+			(xy 77.47 68.58) (xy 77.47 66.04)
+		)
+		(stroke
+			(width 0)
+			(type default)
+		)
+	)
+	(wire
+		(pts
+			(xy 93.98 66.04) (xy 99.06 66.04)
+		)
+		(stroke
+			(width 0)
+			(type default)
+		)
+	)
+	(junction
+		(at 77.47 66.04)
+		(diameter 0)
+		(color 0 0 0 0)
+	)
+	(no_connect
+		(at 93.98 68.58)
+	)
 )

Commit message: C10 (entrada do U5 MCP1824T) 1 uF -> 10 uF/50 V 1206, o datasheet pede 1-10 uF
- DS22070A p.17: 'a typical input capacitance value of 1 uF to 10 uF'; o 1 uF/50 V dava
  0,80 uF a 5 V no pior caso. Novo: C3216X5R1H106K160AB, o mesmo de C4/C8/C31/C32
  (7,0 uF a 5 V). PCB: clone do C4 a 3,5 mm do U5.
- ERC 0; DRC 0 erros, paridade 0. BOM preliminar e PDF regenerados.

Co-Authored-By: Claude Opus 5.5 (1M context) <noreply@anthropic.com>
Claude-Session: https://claude.ai/code/session_01KPnkiJQKrkjgRqqw9M78ie
Parts:
- C10: value 1uF/50V -> 10uF/50V; footprint EBM2_V5:0603C -> EBM2_V5:C_1206_3216Metric; MPN C1608X7R1H105K080AB -> C3216X5R1H106K160AB
Changed lines of the file:
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@@
 			)
 		)
-		(property "Value" "1uF/50V"
+		(property "Value" "10uF/50V"
 			(at 68.58 71.12 0)
 			(show_name no)
@@
 			)
 		)
-		(property "Footprint" "EBM2_V5:0603C"
+		(property "Footprint" "EBM2_V5:C_1206_3216Metric"
 			(at 71.12 69.85 0)
 			(hide yes)
@@
 			)
 		)
-		(property "Description" "Entrada do MCP1824S"
+		(property "Description" "Entrada do MCP1824T: 10 uF/50 V 1206 (28-09-2026). DS22070A p.17 pede 1-10 uF; o 1 uF dava 0,80 uF a 5 V"
 			(at 71.12 69.85 0)
 			(hide yes)
@@
 			)
 		)
-		(property "MPN" "C1608X7R1H105K080AB"
+		(property "MPN" "C3216X5R1H106K160AB"
 			(at 71.12 69.85 0)
 			(hide yes)
